Commit message: add the projection node and corresponding dependency settings

File: jsk_mbzirc_tasks/urdf/hawk.urdf.xacro (robot description, xacro)
@@ -43,6 +43,6 @@
   <!-- Downward facing camera -->
   <xacro:include filename="$(find hector_sensors_description)/urdf/generic_camera.urdf.xacro" />
-  <xacro:generic_camera name="downward_cam" parent="base_link" ros_topic="camera/image" cam_info_topic="camera/camera_info" update_rate="20" res_x="1600" res_y="1200" image_format="R8G8B8" hfov="170">
-    <origin xyz="0.0 0.0 -0.08" rpy="0 ${M_PI/2} 0"/> <!--TODO: modified the position, temporarily right now -->
+  <xacro:generic_camera name="downward_cam" parent="base_link" ros_topic="camera/image" cam_info_topic="camera/camera_info" update_rate="20" res_x="1600" res_y="1200" image_format="R8G8B8" hfov="160">
+    <origin xyz="0.0 0.0 -0.2" rpy="0 ${M_PI/2} 0"/> <!--TODO: modified the position, temporarily right now -->
   </xacro:generic_camera>
   <!-- Sonar height sensor, TODO-> change to laser sensor -->

Commit message: finish task3 simulation demo

File: jsk_mbzirc_tasks/urdf/hawk.urdf.xacro (robot description, xacro)
@@ -44,5 +44,5 @@
   <xacro:include filename="$(find hector_sensors_description)/urdf/generic_camera.urdf.xacro" />
   <xacro:generic_camera name="downward_cam" parent="base_link" ros_topic="camera/image" cam_info_topic="camera/camera_info" update_rate="10" res_x="640" res_y="480" image_format="R8G8B8" hfov="120">
-    <origin xyz="0.0 0.0 -0.2" rpy="0 ${M_PI/2} 0"/> <!--TODO: modified the position, temporarily right now -->
+    <origin xyz="0.0 0.0 -0.05" rpy="0 ${M_PI/2} 0"/> <!--TODO: modified the position, temporarily right now -->
   </xacro:generic_camera>
   <!-- Sonar height sensor, TODO-> change to laser sensor -->
